File: trackpad_R2/trackpad_R2.kicad_pcb (KiCad board)
At the start: 2 copper layers, 107 x 89.2 mm, 29 parts, among them J1 Conn_01x09, U1 74HC4051, U2 74HC4051, U3 74HC4051

Commit message: progress
Parts:
- removed J1: Conn_01x09, Connector_PinHeader_2.54mm:PinHeader_1x09_P2.54mm_Horizontal
- removed TP1: ~, trackpads:trackpad_15x9_100mm_60mm
- added R25: R, Resistor_SMD:R_0805_2012Metric_Pad1.20x1.40mm_HandSolder, F.Cu at (125.2, 3.15)
- added R26: R, Resistor_SMD:R_0805_2012Metric_Pad1.20x1.40mm_HandSolder, F.Cu at (125.2, 6.11)
- added R27: R, Resistor_SMD:R_0805_2012Metric_Pad1.20x1.40mm_HandSolder, F.Cu at (125.2, 9.05)
- added R28: R, Resistor_SMD:R_0805_2012Metric_Pad1.20x1.40mm_HandSolder, F.Cu at (125.2, 12.0)
- added R29: R, Resistor_SMD:R_0805_2012Metric_Pad1.20x1.40mm_HandSolder, F.Cu at (125.2, 15.0)
- added R30: R, Resistor_SMD:R_0805_2012Metric_Pad1.20x1.40mm_HandSolder, F.Cu at (125.2, 17.9)
- added R31: R, Resistor_SMD:R_0805_2012Metric_Pad1.20x1.40mm_HandSolder, F.Cu at (125.2, 20.9)
- added R32: R, Resistor_SMD:R_0805_2012Metric_Pad1.20x1.40mm_HandSolder, F.Cu at (125.2, 23.8)
- added TP2: ~, trackpads:trackpad_20x12_130mm_78mm, F.Cu at (99.2, 54.9)
- added U4: STM32F303CCTx, Package_QFP:LQFP-48_7x7mm_P0.5mm, F.Cu at (63.8, 43.3)
- added U5: LM1117MP-3.3, Package_TO_SOT_SMD:SOT-223-3_TabPin2, F.Cu at (83.2, 45.2)
- added U6: 74HC4051, Package_SO:SOIC-16_3.9x9.9mm_P1.27mm, F.Cu at (140.0, 47.5)
- added Y1: 8MHz, Oscillator:Oscillator_DIP-14, F.Cu at (73.0, 25.4)
- R1, R10, R11, R12, R13, R14, R15, R16, R17, R18, R19, R2, R20, R21, R22, R23, R24, R3, R4, R5, R6, R7, R8, R9, U1, U2, U3: moved to F.Cu
- moved R7 148.3 mm to (194.1, 32.6), turned to 0 degrees
- moved R8 147.1 mm to (194.1, 35.5)
- moved R5 141.5 mm to (189.4, 44.4), turned to 0 degrees
- moved R6 140.0 mm to (189.4, 47.3), turned to 0 degrees
- moved R1 130.6 mm to (189.4, 32.6)
- moved R2 130.4 mm to (189.4, 35.5)
- moved R3 130.1 mm to (189.4, 38.5)
- moved R4 128.1 mm to (189.4, 41.4)
- moved R13 121.7 mm to (198.9, 32.6), turned to 0 degrees
- moved R15 119.5 mm to (198.9, 38.5), turned to 0 degrees
- moved R14 119.2 mm to (198.9, 35.5), turned to 0 degrees
- moved R16 118.3 mm to (198.9, 41.4), turned to 0 degrees
- moved R9 101.8 mm to (194.1, 38.5)
- moved R10 101.6 mm to (194.1, 41.4)
- moved R11 101.3 mm to (194.1, 44.4)
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Routing:
- net /S0: track 125.1 -> 0.00 mm, vias 4 -> 0
- net /S1: track 120.0 -> 0.00 mm, vias 4 -> 0
- net /S2: track 118.2 -> 0.00 mm, vias 4 -> 0
- net VCC: track 115.7 -> 0.00 mm, vias 5 -> 0
- net /A: track 93.6 -> 0.00 mm, vias 4 -> 0
- net /X14: track 75.6 -> 0.00 mm
- net /X11: track 75.5 -> 0.00 mm
- net /X0: track 75.2 -> 0.00 mm
- net /X12: track 75.2 -> 0.00 mm
- net /X4: track 74.8 -> 0.00 mm
- net /X13: track 74.5 -> 0.00 mm
- net /X5: track 72.4 -> 0.00 mm
- net /X1: track 70.1 -> 0.00 mm
- net /X3: track 69.8 -> 0.00 mm
- net /X2: track 68.0 -> 0.00 mm
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Other:
- board size 107 x 89.2 mm -> 142.5 x 105 mm
- board text removed: "Matrix: 15x9 Size: ~100x60mm"
- board text removed: "Trackpad_M2"

Commit message: progres
Parts:
- removed R10, R11, R12, R13, R14, R15, R16, R17, R18, R19, R20, R21, R22, R23, R24, R25, R26, R27, R28, R29, R30, R31, R32, R6, R7, R8, R9: R, Resistor_SMD:R_0805_2012Metric_Pad1.20x1.40mm_HandSolder
- removed TP2: ~, trackpads:trackpad_20x12_130mm_78mm
- removed U1: 74HC4051, Package_SO:SOIC-16_3.9x9.9mm_P1.27mm
- added C1: 10uF, Capacitor_SMD:C_0805_2012Metric, B.Cu at (92.5, 45.2)
- added C2: 10uF, Capacitor_SMD:C_0805_2012Metric, B.Cu at (86.2, 45.2)
- added C3: 100nF, Capacitor_SMD:C_0603_1608Metric_Pad1.08x0.95mm_HandSolder, B.Cu at (114.4, 42.7)
- added C4: 15pF, Capacitor_SMD:C_0603_1608Metric_Pad1.08x0.95mm_HandSolder, B.Cu at (131.6, 46.1)
- added C5: 15pF, Capacitor_SMD:C_0603_1608Metric_Pad1.08x0.95mm_HandSolder, B.Cu at (132.0, 50.0)
- added C6: 100nF, Capacitor_SMD:C_0603_1608Metric_Pad1.08x0.95mm_HandSolder, B.Cu at (123.5, 53.9)
- added C7: 100nF, Capacitor_SMD:C_0603_1608Metric_Pad1.08x0.95mm_HandSolder, B.Cu at (111.6, 49.1)
- added C8: 100nF, Capacitor_SMD:C_0603_1608Metric_Pad1.08x0.95mm_HandSolder, B.Cu at (125.4, 47.5)
- added D1: LED, LED_SMD:LED_1206_3216Metric_ReverseMount_Hole1.8x2.4mm, B.Cu at (101.0, 51.2)
- added J1: USB_C_Receptacle_USB2.0_16P, Connector_USB:USB_C_Receptacle_GCT_USB4105-xx-A_16P_TopMnt_Horizontal, B.Cu at (101.0, 43.5)
- added Q1: NPN, Package_TO_SOT_SMD:SOT-323_SC-70, B.Cu at (95.8, 51.2)
- added SW1: SW_Omron_B3FS, Button_Switch_SMD:SW_Push_1P1T_NO_CK_KMR2, B.Cu at (126.0, 43.5)
- added TP1: ~, trackpads:trackpad_24x14_132mm_77mm, F.Cu at (99.0, 55.0)
- added U7: STM32F303CCTx, Package_QFP:LQFP-48_7x7mm_P0.5mm, B.Cu at (118.5, 48.2)
- added U8: AP2112K-3.3, Package_TO_SOT_SMD:SOT-23-5, B.Cu at (89.2, 45.2)
- R1, R2: value R -> 5.1K; footprint Resistor_SMD:R_0805_2012Metric_Pad1.20x1.40mm_HandSolder -> Resistor_SMD:R_0603_1608Metric_Pad0.98x0.95mm_HandSolder; moved to B.Cu
- R3: value R -> 110; footprint Resistor_SMD:R_0805_2012Metric_Pad1.20x1.40mm_HandSolder -> Resistor_SMD:R_0603_1608Metric_Pad0.98x0.95mm_HandSolder; moved to B.Cu
- R4: value R -> 10K; footprint Resistor_SMD:R_0805_2012Metric_Pad1.20x1.40mm_HandSolder -> Resistor_SMD:R_0603_1608Metric_Pad0.98x0.95mm_HandSolder; moved to B.Cu
- R5: value R -> 4.7K; footprint Resistor_SMD:R_0805_2012Metric_Pad1.20x1.40mm_HandSolder -> Resistor_SMD:R_0603_1608Metric_Pad0.98x0.95mm_HandSolder; moved to B.Cu
- U2, U3, U6: moved to B.Cu
- U4: value STM32F303CCTx -> 74HC4051; footprint Package_QFP:LQFP-48_7x7mm_P0.5mm -> Package_SO:SOIC-16_3.9x9.9mm_P1.27mm; moved to B.Cu
- U5: value LM1117MP-3.3 -> 74HC4051; footprint Package_TO_SOT_SMD:SOT-223-3_TabPin2 -> Package_SO:SOIC-16_3.9x9.9mm_P1.27mm; moved to B.Cu
- Y1: value 8MHz -> Crystal; footprint Oscillator:Oscillator_DIP-14 -> Crystal:Crystal_SMD_Abracon_ABM8G-4Pin_3.2x2.5mm; moved to B.Cu
- moved R5 95.9 mm to (93.7, 51.5), turned to 90 degrees
- moved R1 95.6 mm to (94.5, 44.5), turned to -90 degrees
- moved R3 92.5 mm to (97.8, 51.5), turned to 90 degrees
- moved U4 82.6 mm to (146.0, 51.0), turned to -90 degrees
- moved R2 82.4 mm to (107.5, 44.5), turned to -90 degrees
- moved U2 65.6 mm to (57.0, 51.0), turned to -90 degrees
- moved Y1 61.3 mm to (130.0, 48.0), turned to -45 degrees
- moved R4 56.9 mm to (132.5, 42.8), turned to 180 degrees
- moved U5 42.5 mm to (41.0, 51.0), turned to -90 degrees
- moved U3 24.3 mm to (73.5, 51.0), turned to -90 degrees
- moved U6 22.3 mm to (162.0, 51.0), turned to -90 degrees
Connections:
- R1 pad 1: Net-(U1-A0) -> GND
- R1 pad 2: /Y3 -> Net-(J1-CC1)
- R2 pad 1: Net-(U1-A1) -> GND
- R2 pad 2: /X3 -> Net-(J1-CC2)
- R3 pad 2: /Y2 -> Net-(D1-A)
- R4 pad 1: Net-(U1-A3) -> GND
- R4 pad 2: /X4 -> Net-(U7-BOOT0)
- R5 pad 2: /X2 -> /LED
- U2 pad 1: Net-(U2-A4) -> /RX3
- U2 pad 10: /S1 -> /SX1
- U2 pad 11: /S0 -> /SX0
- U2 pad 12: Net-(U2-A3) -> /RX7
- U2 pad 13: Net-(U2-A0) -> /RX6
- U2 pad 14: Net-(U2-A1) -> /RX5
- U2 pad 15: Net-(U2-A2) -> /RX4
- U2 pad 16: VCC -> +3.3V
- U2 pad 2: Net-(U2-A6) -> /RX2
- U2 pad 3: /A -> /M_OUT
- U2 pad 4: Net-(U2-A7) -> /RX1
- U2 pad 5: Net-(U2-A5) -> /RX0
- U2 pad 6: /E1 -> /E0
- U2 pad 9: /S2 -> /SX2
- U3 pad 1: Net-(U3-A4) -> /RX15
- U3 pad 10: /S1 -> /SX1
- U3 pad 11: /S0 -> /SX0
- U3 pad 12: Net-(U3-A3) -> /RX11
- U3 pad 13: Net-(U3-A0) -> /RX10
- U3 pad 14: Net-(U3-A1) -> /RX9
- U3 pad 15: Net-(U3-A2) -> /RX8
- U3 pad 16: VCC -> +3.3V
- U3 pad 2: Net-(U3-A6) -> /RX14
- U3 pad 3: /A -> /M_OUT
- U3 pad 4: Net-(U3-A7) -> /RX13
- U3 pad 5: Net-(U3-A5) -> /RX12
- U3 pad 6: /E2 -> /E1
- U3 pad 9: /S2 -> /SX2
- U4 pad 1: unconnected-(U4-VBAT-Pad1) -> /RX19
- U4 pad 10: unconnected-(U4-PA0-Pad10) -> /SX1
- U4 pad 11: unconnected-(U4-PA1-Pad11) -> /SX0
- U4 pad 12: unconnected-(U4-PA2-Pad12) -> /RX23
- U4 pad 13: unconnected-(U4-PA3-Pad13) -> /RX22
- U4 pad 14: unconnected-(U4-PA4-Pad14) -> /RX21
- U4 pad 15: unconnected-(U4-PA5-Pad15) -> /RX20
- U4 pad 16: unconnected-(U4-PA6-Pad16) -> +3.3V
- U4 pad 2: unconnected-(U4-PC13-Pad2) -> /RX18
- U4 pad 3: unconnected-(U4-PC14-Pad3) -> /M_OUT
- U4 pad 4: unconnected-(U4-PC15-Pad4) -> /RX17
- U4 pad 5: Net-(U4-PF0) -> /RX16
- U4 pad 6: Net-(U4-PF1) -> /E2
- U4 pad 7: unconnected-(U4-NRST-Pad7) -> GND
- U4 pad 8: unconnected-(U4-VSSA-Pad8) -> GND
- U4 pad 9: unconnected-(U4-VDDA-Pad9) -> /SX2
- U5 pad 1: unconnected-(U5-GND-Pad1) -> /TX6
- U5 pad 2: unconnected-(U5-VO-Pad2) -> /TX8
- U5 pad 3: unconnected-(U5-VI-Pad3) -> /M_IN
- U6 pad 1: Net-(U6-A4) -> /TX13
- U6 pad 10: /S1 -> /SY1
- U6 pad 11: /S0 -> /SY0
- U6 pad 12: Net-(U6-A3) -> unconnected-(U6-A3-Pad12)
- U6 pad 13: Net-(U6-A0) -> /TX5
- U6 pad 14: Net-(U6-A1) -> /TX3
- U6 pad 15: Net-(U6-A2) -> /TX1
- U6 pad 16: VCC -> +3.3V
- U6 pad 2: Net-(U6-A6) -> /TX11
- U6 pad 3: /A -> /M_IN
- U6 pad 4: Net-(U6-A7) -> /TX9
- U6 pad 5: Net-(U6-A5) -> /TX7
- U6 pad 6: /E3 -> /E4
- U6 pad 9: /S2 -> /SY2
- Y1 pad 1: Net-(U4-PF1) -> /Crystal_IN
Routing:
- net /M_IN: track 0.00 -> 147.9 mm, vias 0 -> 2
- net /M_OUT: track 0.00 -> 141.1 mm
- net /RX15: track 0.00 -> 137.7 mm
- net /RX14: track 0.00 -> 130.7 mm
- net /RX13: track 0.00 -> 122.2 mm
- net /RX12: track 0.00 -> 115.0 mm
- net /RX16: track 0.00 -> 110.3 mm
- net /RX0: track 0.00 -> 108.3 mm
- net /TX13: track 0.00 -> 105.4 mm
- net /RX11: track 0.00 -> 103.6 mm
- net /RX17: track 0.00 -> 103.1 mm
- net /RX1: track 0.00 -> 101.1 mm
- net /RX10: track 0.00 -> 99.3 mm
- net /RX7: track 0.00 -> 98.3 mm
- net /RX23: track 0.00 -> 98.2 mm
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Other:
- board size 142.5 x 105 mm -> 146 x 100.2 mm
- board text added: "RX0"
- board text added: "RX0-7"
- board text added: "RX1"
- board text added: "RX10"
- board text added: "RX11"
- board text added: "RX12"
- board text added: "RX13"
- board text added: "RX14"
- board text added: "RX15"
- board text added: "RX16"
- board text added: "RX16-23"
- board text added: "RX17"
- board text added: "RX18"
- board text added: "RX19"
- board text added: "RX2"
- board text added: "RX20"
- board text added: "RX21"
- board text added: "RX22"
- board text added: "RX23"
- board text added: "RX3"
- board text added: "RX4"
- board text added: "RX5"
- board text added: "RX6"
- board text added: "RX7"
- board text added: "RX8"
- board text added: "RX8-15"
- board text added: "RX9"
- board text added: "TX-I"
- board text added: "TX-II"
- board text added: "TX0"
- board text added: "TX1"
- board text added: "TX10"
- board text added: "TX11"
- board text added: "TX12"
- board text added: "TX13"
- board text added: "TX2"
- board text added: "TX3"
- board text added: "TX4"
- board text added: "TX5"
- board text added: "TX6"
- board text added: "TX7"
- board text added: "TX8"
- board text added: "TX9"
- board text added: "Zäni"

Commit message: Progress + images
Parts:
- moved C6 0.45 mm to (123.5, 54.4)
Connections:
- U7 pad 17: unconnected-(U7-PA7-Pad17) -> /SX2
- U7 pad 18: /SX2 -> /SX1
- U7 pad 19: /SX1 -> /SX0
- U7 pad 20: /SX0 -> /SY2
- U7 pad 21: /SY2 -> /SY1
- U7 pad 22: /SY1 -> /SY0
- U7 pad 25: /SY0 -> unconnected-(U7-PB12-Pad25)
- U7 pad 39: /E0 -> /E3
- U7 pad 40: /E1 -> /E0
- U7 pad 41: /E2 -> /E1
- U7 pad 42: /E3 -> unconnected-(U7-PB6-Pad42)
- U7 pad 45: unconnected-(U7-PB8-Pad45) -> /E2
Routing:
- net +3.3V: track 80.0 -> 229.6 mm, vias 4 -> 13
- net /SY2: track 35.5 -> 137.2 mm, vias 1 -> 3
- net /SY1: track 36.2 -> 135.6 mm, vias 1 -> 3
- net /SY0: track 45.9 -> 134.1 mm, vias 1 -> 3
- net /SX2: track 25.6 -> 106.2 mm, vias 3 -> 4
- net /SX1: track 23.5 -> 103.6 mm, vias 3 -> 4
- net /SX0: track 21.3 -> 101.1 mm, vias 3 -> 4
- net /E1: track 0.00 -> 58.0 mm, vias 0 -> 3
- net /E4: track 0.00 -> 49.8 mm, vias 0 -> 2
- net /E0: track 30.1 -> 72.6 mm, vias 1 -> 2
- net /E3: track 49.4 -> 88.1 mm, vias 1 -> 2
- net /E2: track 2.06 -> 30.8 mm, vias 1 -> 2
- net Net-(J1-CC1): track 9.97 -> 8.23 mm, vias 2 -> 0
- net /M_OUT: track 141.1 -> 142.5 mm
- net /M_IN: track 147.9 -> 146.6 mm
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